File: Hardware/Camera/Camera.kicad_sch (KiCad schematic)
At the start: 5 parts

Commit message: Finished initial positioning!
Parts:
- added C10, C11, C15: 10u, Capacitor_SMD:C_1206_3216Metric, symbol Device:C_Small
- added C12, C17, C19: 1u, Capacitor_SMD:C_0402_1005Metric, symbol Device:C_Small
- added C13, C16: 10p, Capacitor_SMD:C_0402_1005Metric, symbol Device:C_Small
- added C14: 10n, Capacitor_SMD:C_0402_1005Metric, symbol Device:C_Small
- added C18: 10n, Capacitor_SMD:C_1206_3216Metric, symbol Device:C_Small
- added C3: 4u7, Capacitor_SMD:C_0603_1608Metric, symbol Device:C_Small
- added C4, C5, C6, C8, C9: 100n, Capacitor_SMD:C_0402_1005Metric, symbol Device:C_Small
- added C7: 1n, Capacitor_SMD:C_0603_1608Metric, symbol Device:C_Small
- added D1, D2: B5819W, Diode_SMD:D_SOD-123, symbol Device:D_Schottky
- added D3: USBLC6-2SC6, digikey-footprints:SOT23-6L, symbol dk_TVS-Diodes:USBLC6-2SC6
- added D4: BLUE, LED_SMD:LED_0603_1608Metric, symbol Device:LED
- added D5, D6: RED, LED_SMD:LED_0603_1608Metric, symbol Device:LED
- added F1: 250 mA, Fuse:Fuse_1206_3216Metric, symbol Device:Polyfuse
- added FB1: 600 @ 600MHz, Inductor_SMD:L_0805_2012Metric, symbol Device:FerriteBead
- added GND1: MP2359DJ, Package_TO_SOT_SMD:SOT-23-6, symbol Troy:MP2359DJ
- added H1, H2, H3, H4: MountingHole_Pad, MountingHole:MountingHole_4.3mm_M4_Pad_Via, symbol Mechanical:MountingHole_Pad
- added J1: Power, TerminalBlock_Phoenix:TerminalBlock_Phoenix_PT-1,5-2-3.5-H_1x02_P3.50mm_Horizontal, symbol Connector:Screw_Terminal_01x02
- added J2: ICC Out, TerminalBlock_Phoenix:TerminalBlock_Phoenix_PT-1,5-4-3.5-H_1x04_P3.50mm_Horizontal, symbol Connector:Screw_Terminal_01x04
- added J3: USB_B_Mini, Connector_USB:USB_Micro-B_Molex-105133-0031, symbol Connector:USB_B_Mini
- added J4: SWDIO, Connector_PinSocket_1.27mm:PinSocket_2x05_P1.27mm_Vertical_SMD, symbol Connector_Generic_MountingPin:Conn_02x05_Odd_Even_MountingPin
- added J5: Header Pins, Connector_PinHeader_1.27mm:PinHeader_2x11_P1.27mm_Vertical_SMD, symbol Connector_Generic_MountingPin:Conn_02x11_Odd_Even_MountingPin
- added J6: Camer Interface, Connector_PinHeader_1.00mm:PinHeader_1x24_P1.00mm_Vertical_SMD_Pin1Left, symbol Connector:Conn_01x24_Female
- added L1: 10u, Inductor_SMD:L_6.3x6.3_H3, symbol Device:L
- added L2: 39n, Inductor_SMD:L_0603_1608Metric, symbol Device:L_Small
- added Q1: AO3401A, Custom:AO3401A, symbol dk_Transistors-FETs-MOSFETs-Single:AO3401A
- added R1: 100k, Resistor_SMD:R_0603_1608Metric, symbol Device:R_Small
- added R10: 20, Resistor_SMD:R_0402_1005Metric, symbol Device:R_Small
- added R11: 47k, Resistor_SMD:R_0603_1608Metric, symbol Device:R_Small
- added R12: 15k, Resistor_SMD:R_0603_1608Metric, symbol Device:R_Small
- added R13: 270, Resistor_SMD:R_0603_1608Metric, symbol Device:R_Small
- added R14, R16, R19: 240, Resistor_SMD:R_0603_1608Metric, symbol Device:R_Small
- added R15: 47, Resistor_SMD:R_0603_1608Metric, symbol Device:R_Small
- added R18: 10, Resistor_SMD:R_0603_1608Metric, symbol Device:R_Small
- added R2: 68k, Resistor_SMD:R_0603_1608Metric, symbol Device:R_Small
- added R20: 2k, Resistor_SMD:R_0603_1608Metric, symbol Device:R_Small
- added R3, R4, R5: 1m, Resistor_SMD:R_0603_1608Metric, symbol Device:R_Small
- added R6, R7: 1k5, Resistor_SMD:R_0603_1608Metric, symbol Device:R_Small
- added R8, R9: 4k7, Resistor_SMD:R_0402_1005Metric, symbol Device:R_Small
- added U2, U3: LM317L_SOT-89, Package_TO_SOT_SMD:SOT-89-3, symbol Regulator_Linear:LM317L_SOT-89
- added Y1: 16MHz, Crystal:Crystal_SMD_3225-4Pin_3.2x2.5mm, symbol Device:Crystal_GND24_Small
- C1, C2: renamed from C?; footprint (none) -> Capacitor_SMD:C_0603_1608Metric
- R17: renamed from R?; footprint (none) -> Resistor_SMD:R_0402_1005Metric
- SW1: renamed from SW?; footprint (none) -> Button_Switch_SMD:SW_SPDT_PCM12
- gave numbers to parts that had none: 1
Connections:
- net +3.3VA: now also C12.1, C14.1, L2.2, U2.3 (VI)
- net +3V3: now also C11.1, C15.1, C3.1, C4.1, C5.1, C6.1, C8.1, C9.1, D6.2 (A), J2.1 (Pin_1), J4.1 (Pin_1), J5.1 (Pin_1), J5.22 (Pin_22), J6.11 (Pin_11), L1.2, L2.1, R11.1, R8.1, R9.1, U3.3 (VI)
- net CAM_PWDN: now also J6.8 (Pin_8)
- net CAM_STROBE: now also J6.1 (Pin_1)
- net DCMI0: now also J6.24 (Pin_24)
- net DCMI1: now also J6.23 (Pin_23)
- net DCMI2: now also J6.19 (Pin_19)
- net DCMI3: now also J6.21 (Pin_21)
- net DCMI4: now also J6.22 (Pin_22)
- net DCMI5: now also J6.20 (Pin_20)
- net DCMI6: now also J6.18 (Pin_18)
- net DCMI7: now also J6.16 (Pin_16)
- net DCMI8: now also J6.14 (Pin_14)
- net DCMI9: now also J6.12 (Pin_12)
- net DCMI_HSYNC: now also J6.9 (Pin_9)
- net DCMI_PIXCLK: now also J6.17 (Pin_17)
- net DCMI_VSYNC: now also J6.7 (Pin_7)
- net GND: now also C10.2, C11.2, C12.2, C13.2, C14.2, C15.2, C16.2, C17.2, C19.2, C3.2, C4.2, C5.2, C6.2, C7.2, C8.2, C9.2, D2.2 (A), D3.2, GND1.2 (GND), H1.1, H2.1, H3.1, H4.1, J1.2 (Pin_2), J2.2 (Pin_2), J3.5 (GND), J4.3 (Pin_3), J4.5 (Pin_5), J4.9 (Pin_9), J5.2 (Pin_2), J5.21 (Pin_21), J6.15 (Pin_15), J6.2 (Pin_2), Q1.1 (G), R13.2, R15.2, R18.2, R2.2, R20.2, R5.2, R6.2, R7.2, Y1.2, Y1.4
- net GPIO0: now also J5.10 (Pin_10)
- net GPIO1: now also J5.11 (Pin_11)
- net GPIO2: now also J5.12 (Pin_12)
- net HSE_IN: now also C13.1, Y1.1
- net HSE_OUT: now also R10.1
- net I2C2_SCL: now also J5.7 (Pin_7), J6.5 (Pin_5), R8.2
- net I2C2_SDA: now also J5.9 (Pin_9), J6.3 (Pin_3), R9.2
- net LED_STATUS: now also D4.2 (A)
- net LED_STATUS_2: now also D5.2 (A)
- net NRST: now also J4.10 (Pin_10)
- net RCC_MCO_1: now also J5.19 (Pin_19)
- net RCC_MCO_2: now also J6.13 (Pin_13)
- net SPI2_MISO: now also J5.6 (Pin_6)
- net SPI2_MOSI: now also J5.8 (Pin_8)
- net SPI2_SCK: now also J5.4 (Pin_4)
- net SWCLK: now also J4.4 (Pin_4)
- net SWDIO: now also J4.2 (Pin_2)
- net SWO: now also J4.6 (Pin_6)
- net USART3_RX: now also J5.20 (Pin_20)
- net USART3_TX: now also J5.18 (Pin_18)
- net USART6_RX: now also J2.4 (Pin_4)
- net USART6_TX: now also J2.3 (Pin_3)
- net USB_D+: now also D3.6
- net USB_D-: now also D3.4
- net USART2_TX: now reaches U1.36 (PA2)
- net USART2_TX: now also J5.3 (Pin_3)
- net USART2_RX: now reaches U1.37 (PA3)
- net USART2_RX: now also J5.5 (Pin_5)
- net GPIO3: now reaches U1.79 (PD10)
- net GPIO3: now also J5.13 (Pin_13)
- net GPIO4: now reaches U1.80 (PD11)
- net GPIO4: now also J5.14 (Pin_14)
- net GPIO5: now reaches U1.81 (PD12)
- net GPIO5: now also J5.15 (Pin_15)
- net GPIO6: now reaches U1.82 (PD13)
- net GPIO6: now also J5.16 (Pin_16)
- net GPIO7: now reaches U1.85 (PD14)
- net GPIO7: now also J5.17 (Pin_17)
- net BAT_GPIO_IN renamed BAT_A_IN
- net BAT_A_IN: now also C7.1, R4.2, R5.1
- net CAM_EXPST_B: no longer names the net of U1.90 (PG5)
- net CAM_FREX renamed CAM_RESET
- net CAM_RESET: now also J6.6 (Pin_6)
- net JTDI: no longer names the net of U1.110 (PA15)
- net JTRST: no longer names the net of U1.134 (PB4)
- new net: R12.2, R13.1
- new net: R14.1, R16.2, U2.1 (ADJ)
- new net: R14.2, R15.1
- new net: D5.1 (K), R7.1
- new net: D1.1 (K), FB1.1, Q1.2 (S), R3.1
- new net: R3.2, R4.1
- new net: R18.1, R19.2, U3.1 (ADJ)
- new net: F1.2, Q1.3 (D)
- new net: D3.3, J3.2 (D-)
- new net: D3.1, J3.3 (D+)
- new net: D6.1 (K), R20.1
- new net: C16.1, R10.2, Y1.3
- new net: D4.1 (K), R6.1
- new net +5V: D1.2 (A), D3.5, J3.1 (VBUS)
- new net +9V: F1.1, J1.1 (Pin_1)
- new net AVCC_2V8: C17.1, J6.4 (Pin_4), R16.1, U2.2 (VO)
- new net BUCK_BST: C18.1, GND1.1 (BST)
- new net BUCK_EN: GND1.4 (EN), R1.2, R2.1
- new net BUCK_FB: GND1.3 (FB), R11.2, R12.1
- new net BUCK_IN: C10.1, FB1.2, GND1.5 (IN), R1.1
- new net BUCK_SW: C18.2, D2.1 (K), GND1.6 (SW), L1.1
- new net VCC_1V3: C19.1, J6.10 (Pin_10), R19.1, U3.2 (VO)
- no-connect marks 72 -> 73
Other:
- note added: "1.24-1.36V (1.3V) @ 30-40mA"
- note added: "1.71-3.3V (2.8) @ 6-15mA"
- note added: "2.5-3.0V (2.8V) @ 30-40mA"
- note added: "Analog Filtering"
- note added: "Connectors"
- note added: "Digital Ground"
- note added: "Divide 9v input to below 6v so that the buck converter turns on"
- note added: "HREF"
- note added: "JTDI"
- note added: "MCLK"
- note added: "Makes a 49.9 / 16.2 Ohm voltage divider"
- note added: "PCLK"
- note added: "Power Circuitry"
- note added: "STM32 Microcontroller"
- moved on the sheet: C1, C2, R17, SW1, U1

Commit message: Small improvements for pre-routing
Changed lines of the file:
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@@
     (stroke (width 0) (type default) (color 0 0 0 0))
   )
+  (wire (pts (xy 274.32 105.41) (xy 290.83 105.41))
+    (stroke (width 0) (type default) (color 0 0 0 0))
+  )
   (wire (pts (xy 203.2 179.07) (xy 209.55 179.07))
     (stroke (width 0) (type default) (color 0 0 0 0))
@@
     (stroke (width 0) (type default) (color 0 0 0 0))
   )
-  (wire (pts (xy 290.83 168.91) (xy 298.704 168.91))
-    (stroke (width 0) (type default) (color 0 0 0 0))
-  )
   (wire (pts (xy 76.2 204.47) (xy 76.2 207.01))
     (stroke (width 0) (type default) (color 0 0 0 0))
@@
     (stroke (width 0) (type default) (color 0 0 0 0))
   )
+  (wire (pts (xy 273.05 125.73) (xy 273.05 128.27))
+    (stroke (width 0) (type default) (color 0 0 0 0))
+  )
   (wire (pts (xy 66.04 59.69) (xy 66.04 57.15))
     (stroke (width 0) (type default) (color 0 0 0 0))
@@
     (stroke (width 0) (type default) (color 0 0 0 0))
   )
+  (wire (pts (xy 273.05 140.97) (xy 273.05 138.43))
+    (stroke (width 0) (type default) (color 0 0 0 0))
+  )
   (wire (pts (xy 147.32 186.69) (xy 153.67 186.69))
     (stroke (width 0) (type default) (color 0 0 0 0))
@@
     (stroke (width 0) (type default) (color 0 0 0 0))
   )
+  (wire (pts (xy 274.32 107.95) (xy 274.32 105.41))
+    (stroke (width 0) (type default) (color 0 0 0 0))
+  )
   (wire (pts (xy 33.02 237.49) (xy 33.02 238.76))
     (stroke (width 0) (type default) (color 0 0 0 0))
@@
     (stroke (width 0) (type default) (color 0 0 0 0))
   )
-  (wire (pts (xy 290.83 175.26) (xy 298.45 175.26))
-    (stroke (width 0) (type default) (color 0 0 0 0))
-  )
   (wire (pts (xy 147.32 191.77) (xy 153.67 191.77))
     (stroke (width 0) (type default) (color 0 0 0 0))
@@
     (stroke (width 0) (type default) (color 0 0 0 0))
   )
+  (wire (pts (xy 273.05 138.43) (xy 290.83 138.43))
+    (stroke (width 0) (type default) (color 0 0 0 0))
+  )
   (wire (pts (xy 63.5 391.16) (xy 63.5 389.89))
     (stroke (width 0) (type default) (color 0 0 0 0))
@@
     (stroke (width 0) (type default) (color 0 0 0 0))
   )
+  (wire (pts (xy 273.05 128.27) (xy 290.83 128.27))
+    (stroke (width 0) (type default) (color 0 0 0 0))
+  )
   (wire (pts (xy 71.12 204.47) (xy 71.12 207.01))
     (stroke (width 0) (type default) (color 0 0 0 0))
@@
     (stroke (width 0) (type default) (color 0 0 0 0))
   )
-  (wire (pts (xy 290.83 181.61) (xy 298.45 181.61))
-    (stroke (width 0) (type default) (color 0 0 0 0))
-  )
   (wire (pts (xy 148.59 303.53) (xy 151.13 303.53))
     (stroke (width 0) (type default) (color 0 0 0 0))
@@
     (effects (font (size 1.27 1.27)) (justify left bottom))
   )
-  (text "1.71-3.3V (2.8) @ 6-15mA" (at 299.974 168.91 0)
+  (text "1.71-3.3V (2.8) @ 6-15mA" (at 295.91 129.286 0)
     (effects (font (size 1.27 1.27)) (justify left bottom))
   )
@@
     )
   )
-  (global_label "CAM_DOVDD" (shape input) (at 290.83 168.91 180) (fields_autoplaced)
-    (effects (font (size 1.27 1.27)) (justify right))
-    (property "Intersheet References" "${INTERSHEET_REFS}" (id 0) (at 277.4102 168.8306 0)
-      (effects (font (size 1.27 1.27)) (justify right) hide)
-    )
-  )
   (global_label "VCC_1V3" (shape input) (at 240.03 58.42 0) (fields_autoplaced)
     (effects (font (size 1.27 1.27)) (justify left))
@@
     )
   )
-  (global_label "CAM_DOVDD" (shape input) (at 290.83 128.27 180) (fields_autoplaced)
-    (effects (font (size 1.27 1.27)) (justify right))
-    (property "Intersheet References" "${INTERSHEET_REFS}" (id 0) (at 277.4102 128.1906 0)
-      (effects (font (size 1.27 1.27)) (justify right) hide)
-    )
-  )
   (global_label "NRST" (shape input) (at 43.18 214.63 180) (fields_autoplaced)
     (effects (font (size 1.27 1.27)) (justify right))
@@
     )
   )
-  (global_label "CAM_GND" (shape input) (at 290.83 175.26 180) (fields_autoplaced)
-    (effects (font (size 1.27 1.27)) (justify right))
-    (property "Intersheet References" "${INTERSHEET_REFS}" (id 0) (at 279.7688 175.1806 0)
-      (effects (font (size 1.27 1.27)) (justify right) hide)
-    )
-  )
   (global_label "SWDIO" (shape input) (at 185.42 124.46 0) (fields_autoplaced)
     (effects (font (size 1.27 1.27)) (justify left))
@@
     )
   )
-  (global_label "CAM_GND" (shape input) (at 290.83 138.43 180) (fields_autoplaced)
-    (effects (font (size 1.27 1.27)) (justify right))
-    (property "Intersheet References" "${INTERSHEET_REFS}" (id 0) (at 279.7688 138.3506 0)
-      (effects (font (size 1.27 1.27)) (justify right) hide)
-    )
-  )
   (global_label "DCMI3" (shape input) (at 43.18 346.71 180) (fields_autoplaced)
     (effects (font (size 1.27 1.27)) (justify right))
@@
     )
   )
-  (global_label "CAM_GNDA" (shape input) (at 290.83 181.61 180) (fields_autoplaced)
-    (effects (font (size 1.27 1.27)) (justify right))
-    (property "Intersheet References" "${INTERSHEET_REFS}" (id 0) (at 278.6802 181.5306 0)
-      (effects (font (size 1.27 1.27)) (justify right) hide)
-    )
-  )
-  (global_label "CAM_GNDA" (shape input) (at 290.83 105.41 180) (fields_autoplaced)
-    (effects (font (size 1.27 1.27)) (justify right))
-    (property "Intersheet References" "${INTERSHEET_REFS}" (id 0) (at 278.6802 105.3306 0)
-      (effects (font (size 1.27 1.27)) (justify right) hide)
-    )
-  )
   (global_label "BUCK_FB" (shape input) (at 171.45 57.15 0) (fields_autoplaced)
     (effects (font (size 1.27 1.27)) (justify left))
@@
     (pin "2")
   )
-  (symbol (lib_id "power:GNDA") (at 298.45 181.61 0) (unit 1)
-    (in_bom yes) (on_board yes)
-    (property "Reference" "#PWR058" (id 0) (at 298.45 187.96 0)
-      (effects (font (size 1.27 1.27)) hide)
-    )
-    (property "Value" "GNDA" (id 1) (at 298.45 185.42 0))
-    (property "Footprint" "" (id 2) (at 298.45 181.61 0)
-      (effects (font (size 1.27 1.27)) hide)
-    )
-    (property "Datasheet" "" (id 3) (at 298.45 181.61 0)
-      (effects (font (size 1.27 1.27)) hide)
-    )
-    (pin "1")
-  )
   (symbol (lib_id "Device:R_Small") (at 163.83 60.96 0) (unit 1)
     (in_bom yes) (on_board yes) (fields_autoplaced)
@@
     (pin "1")
   )
-  (symbol (lib_id "power:+3.3V") (at 298.704 168.91 0) (unit 1)
+  (symbol (lib_id "power:+3.3V") (at 273.05 125.73 0) (unit 1)
     (in_bom yes) (on_board yes) (fields_autoplaced)
-    (property "Reference" "#PWR059" (id 0) (at 298.704 172.72 0)
+    (property "Reference" "#PWR059" (id 0) (at 273.05 129.54 0)
       (effects (font (size 1.27 1.27)) hide)
     )
-    (property "Value" "+3.3V" (id 1) (at 298.704 163.83 0))
-    (property "Footprint" "" (id 2) (at 298.704 168.91 0)
+    (property "Value" "+3.3V" (id 1) (at 273.05 120.65 0))
+    (property "Footprint" "" (id 2) (at 273.05 125.73 0)
       (effects (font (size 1.27 1.27)) hide)
     )
-    (property "Datasheet" "" (id 3) (at 298.704 168.91 0)
+    (property "Datasheet" "" (id 3) (at 273.05 125.73 0)
       (effects (font (size 1.27 1.27)) hide)
     )
@@
     (pin "1")
   )
+  (symbol (lib_id "power:GNDA") (at 274.32 107.95 0) (unit 1)
+    (in_bom yes) (on_board yes)
+    (property "Reference" "#PWR0101" (id 0) (at 274.32 114.3 0)
+      (effects (font (size 1.27 1.27)) hide)
+    )
+    (property "Value" "GNDA" (id 1) (at 274.32 111.76 0))
+    (property "Footprint" "" (id 2) (at 274.32 107.95 0)
+      (effects (font (size 1.27 1.27)) hide)
+    )
+    (property "Datasheet" "" (id 3) (at 274.32 107.95 0)
+      (effects (font (size 1.27 1.27)) hide)
+    )
+    (pin "1")
+  )
   (symbol (lib_id "power:+3.3V") (at 64.77 124.46 0) (unit 1)
     (in_bom yes) (on_board yes) (fields_autoplaced)
@@
     (pin "1")
   )
-  (symbol (lib_id "power:GND") (at 298.45 175.26 0) (unit 1)
+  (symbol (lib_id "power:GND") (at 273.05 140.97 0) (unit 1)
     (in_bom yes) (on_board yes)
-    (property "Reference" "#PWR057" (id 0) (at 298.45 181.61 0)
+    (property "Reference" "#PWR057" (id 0) (at 273.05 147.32 0)
       (effects (font (size 1.27 1.27)) hide)
     )
-    (property "Value" "GND" (id 1) (at 298.45 179.07 0))
-    (property "Footprint" "" (id 2) (at 298.45 175.26 0)
+    (property "Value" "GND" (id 1) (at 273.05 144.78 0))
+    (property "Footprint" "" (id 2) (at 273.05 140.97 0)
       (effects (font (size 1.27 1.27)) hide)
     )
-    (property "Datasheet" "" (id 3) (at 298.45 175.26 0)
+    (property "Datasheet" "" (id 3) (at 273.05 140.97 0)
       (effects (font (size 1.27 1.27)) hide)
     )
@@
       (reference "#PWR057") (unit 1) (value "GND") (footprint "")
     )
-    (path "/9cd3ef15-a2f2-4db4-be67-915a7194db8b"
-      (reference "#PWR058") (unit 1) (value "GNDA") (footprint "")
-    )
     (path "/aef60752-facd-42af-ad13-5c46271e902f"
       (reference "#PWR059") (unit 1) (value "+3.3V") (footprint "")
     )
+    (path "/b142b88f-5214-4eb4-bfeb-5c74e74881c7"
+      (reference "#PWR0101") (unit 1) (value "GNDA") (footprint "")
+    )
     (path "/210047a1-42d1-4806-9f8b-752927a4e656"

Commit message: Optimizing camera placement
Parts:
- J6: footprint Connector_PinHeader_1.00mm:PinHeader_1x24_P1.00mm_Vertical_SMD_Pin1Left -> Lib:SAMTEC_ZF5S-24-01-T-WT
Changed lines of the file:
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@@
       (effects (font (size 1.27 1.27)) (justify left))
     )
-    (property "Footprint" "Connector_PinHeader_1.00mm:PinHeader_1x24_P1.00mm_Vertical_SMD_Pin1Left" (id 2) (at 295.91 130.81 0)
+    (property "Footprint" "Lib:SAMTEC_ZF5S-24-01-T-WT" (id 2) (at 295.91 130.81 0)
       (effects (font (size 1.27 1.27)) hide)
     )
@@
     )
     (path "/701033a6-4188-46b9-b56d-63cc408b62d6"
-      (reference "J6") (unit 1) (value "Camer Interface") (footprint "Connector_PinHeader_1.00mm:PinHeader_1x24_P1.00mm_Vertical_SMD_Pin1Left")
+      (reference "J6") (unit 1) (value "Camer Interface") (footprint "Lib:SAMTEC_ZF5S-24-01-T-WT")
     )
     (path "/788a04c2-6e94-4f16-bd0e-64642763e556"

Commit message: Basic routing done
Parts:
- removed J5: Header Pins, Connector_PinHeader_1.27mm:PinHeader_2x11_P1.27mm_Vertical_SMD, symbol Connector_Generic_MountingPin:Conn_02x11_Odd_Even_MountingPin
- added J5: Breakout, Connector_PinHeader_1.27mm:PinHeader_1x20_P1.27mm_Vertical, symbol Connector_Generic:Conn_01x20
Connections:
- net +3V3: now also J5.20 (Pin_20)
- net GND: now also J5.19 (Pin_19)
- net GPIO0: now also J5.14 (Pin_14)
- net GPIO1: now also J5.13 (Pin_13)
- net GPIO2: now also J5.12 (Pin_12)
- net GPIO3: now also J5.6 (Pin_6)
- net GPIO4: now also J5.5 (Pin_5)
- net GPIO5: now also J5.4 (Pin_4)
- net GPIO6: now also J5.3 (Pin_3)
- net GPIO7: now also J5.2 (Pin_2)
- net I2C2_SCL: now also J5.18 (Pin_18)
- net I2C2_SDA: now also J5.17 (Pin_17)
- net RCC_MCO_1: now also J5.1 (Pin_1)
- net USART2_RX: now also J5.16 (Pin_16)
- net USART2_TX: now also J5.15 (Pin_15)
- net USART3_RX: now also J5.7 (Pin_7)
- net USART3_TX: now also J5.8 (Pin_8)
- no-connect marks 73 -> 75

Commit message: About to re-do layout
Parts:
- added MK1: MIC, Sensor_Audio:Infineon_PG-LLGA-5-1, symbol Sensor_Audio:IM69D130
Connections:
- net AVCC_2V8: now also MK1.2 (VDD)
- net GND: now also MK1.4 (SELECT), MK1.5 (GND)
- net SPI2_MISO: now also MK1.1 (DATA)
- net SPI2_SCK: now also MK1.3 (CLOCK)
Changed lines of the file:
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@@
   (no_connect (at 43.18 377.19))
   (no_connect (at 93.98 139.7))
+  (wire (pts (xy 261.62 187.96) (xy 261.62 185.42))
+    (stroke (width 0) (type default) (color 0 0 0 0))
+  )
   (wire (pts (xy 138.43 58.42) (xy 148.59 58.42))
     (stroke (width 0) (type default) (color 0 0 0 0))
@@
     (stroke (width 0) (type default) (color 0 0 0 0))
   )
+  (wire (pts (xy 261.62 167.64) (xy 261.62 170.18))
+    (stroke (width 0) (type default) (color 0 0 0 0))
+  )
   (wire (pts (xy 60.96 204.47) (xy 60.96 207.01))
     (stroke (width 0) (type default) (color 0 0 0 0))
@@
     (stroke (width 0) (type default) (color 0 0 0 0))
   )
+  (wire (pts (xy 271.78 175.26) (xy 288.29 175.26))
+    (stroke (width 0) (type default) (color 0 0 0 0))
+  )
   (wire (pts (xy 151.13 33.02) (xy 151.13 35.56))
     (stroke (width 0) (type default) (color 0 0 0 0))
@@
     )
   )
+  (global_label "AVCC_2V8" (shape input) (at 261.62 167.64 0) (fields_autoplaced)
+    (effects (font (size 1.27 1.27)) (justify left))
+    (property "Intersheet References" "${INTERSHEET_REFS}" (id 0) (at 273.2255 167.5606 0)
+      (effects (font (size 1.27 1.27)) (justify left) hide)
+    )
+  )
   (global_label "USART3_TX" (shape input) (at 229.87 121.92 180) (fields_autoplaced)
     (effects (font (size 1.27 1.27)) (justify right))
@@
     )
   )
+  (global_label "SPI2_MISO" (shape input) (at 271.78 180.34 0) (fields_autoplaced)
+    (effects (font (size 1.27 1.27)) (justify left))
+    (property "Intersheet References" "${INTERSHEET_REFS}" (id 0) (at 284.0507 180.2606 0)
+      (effects (font (size 1.27 1.27)) (justify left) hide)
+    )
+  )
   (global_label "DCMI_VSYNC" (shape input) (at 290.83 118.11 180) (fields_autoplaced)
     (effects (font (size 1.27 1.27)) (justify right))
@@
     )
   )
+  (global_label "SPI2_SCK" (shape input) (at 271.78 177.8 0) (fields_autoplaced)
+    (effects (font (size 1.27 1.27)) (justify left))
+    (property "Intersheet References" "${INTERSHEET_REFS}" (id 0) (at 283.2041 177.7206 0)
+      (effects (font (size 1.27 1.27)) (justify left) hide)
+    )
+  )
   (global_label "I2C2_SDA" (shape input) (at 43.18 300.99 180) (fields_autoplaced)
     (effects (font (size 1.27 1.27)) (justify right))
@@
     (pin "1")
   )
+  (symbol (lib_id "Sensor_Audio:IM69D130") (at 261.62 177.8 0) (unit 1)
+    (in_bom yes) (on_board yes) (fields_autoplaced)
+    (property "Reference" "MK1" (id 0) (at 252.73 176.5299 0)
+      (effects (font (size 1.27 1.27)) (justify right))
+    )
+    (property "Value" "MIC" (id 1) (at 252.73 179.0699 0)
+      (effects (font (size 1.27 1.27)) (justify right))
+    )
+    (property "Footprint" "Sensor_Audio:Infineon_PG-LLGA-5-1" (id 2) (at 279.4 185.42 0)
+      (effects (font (size 1.27 1.27) italic) hide)
+    )
+    (property "Datasheet" "https://www.infineon.com/dgdl/Infineon-IM69D130-DS-v01_00-EN.pdf?fileId=5546d462602a9dc801607a0e46511a2e" (id 3) (at 261.62 177.8 0)
+      (effects (font (size 1.27 1.27)) hide)
+    )
+    (pin "1")
+    (pin "2")
+    (pin "3")
+    (pin "4")
+    (pin "5")
+  )
   (symbol (lib_id "Device:C_Small") (at 139.7 189.23 0) (unit 1)
     (in_bom yes) (on_board yes) (fields_autoplaced)
@@
     (pin "2")
   )
+  (symbol (lib_id "power:GNDA") (at 261.62 187.96 0) (unit 1)
+    (in_bom yes) (on_board yes)
+    (property "Reference" "#PWR054" (id 0) (at 261.62 194.31 0)
+      (effects (font (size 1.27 1.27)) hide)
+    )
+    (property "Value" "GNDA" (id 1) (at 261.62 191.77 0))
+    (property "Footprint" "" (id 2) (at 261.62 187.96 0)
+      (effects (font (size 1.27 1.27)) hide)
+    )
+    (property "Datasheet" "" (id 3) (at 261.62 187.96 0)
+      (effects (font (size 1.27 1.27)) hide)
+    )
+    (pin "1")
+  )
   (symbol (lib_id "Device:D_Schottky") (at 58.42 22.86 90) (unit 1)
     (in_bom yes) (on_board yes) (fields_autoplaced)
@@
     (pin "1")
   )
+  (symbol (lib_id "power:GNDA") (at 288.29 175.26 0) (unit 1)
+    (in_bom yes) (on_board yes)
+    (property "Reference" "#PWR055" (id 0) (at 288.29 181.61 0)
+      (effects (font (size 1.27 1.27)) hide)
+    )
+    (property "Value" "GNDA" (id 1) (at 288.29 179.07 0))
+    (property "Footprint" "" (id 2) (at 288.29 175.26 0)
+      (effects (font (size 1.27 1.27)) hide)
+    )
+    (property "Datasheet" "" (id 3) (at 288.29 175.26 0)
+      (effects (font (size 1.27 1.27)) hide)
+    )
+    (pin "1")
+  )
   (symbol (lib_id "power:GND") (at 24.13 238.76 0) (unit 1)
     (in_bom yes) (on_board yes) (fields_autoplaced)
@@
       (reference "#PWR053") (unit 1) (value "GND") (footprint "")
     )
+    (path "/2cbb60b3-780c-4df0-85f4-a3eb01190307"
+      (reference "#PWR054") (unit 1) (value "GNDA") (footprint "")
+    )
+    (path "/965f769a-a693-48ab-b5f2-7607ed82b7ee"
+      (reference "#PWR055") (unit 1) (value "GNDA") (footprint "")
+    )
     (path "/92f31037-40e8-4176-8082-8041f0da9201"
       (reference "#PWR056") (unit 1) (value "GND") (footprint "")
@@
       (reference "L2") (unit 1) (value "39n") (footprint "Inductor_SMD:L_0603_1608Metric")
     )
+    (path "/12c7caee-e148-470b-9da2-ccaee29beb5f"
+      (reference "MK1") (unit 1) (value "MIC") (footprint "Sensor_Audio:Infineon_PG-LLGA-5-1")
+    )
     (path "/aa7af968-5118-421d-bd21-75f0ddb649f1"
